Commit message: 3D kinematic upgrade: prismatic lift + ros2_control + anti-explosion spawning
URDF / Kinematics:
- Added lift_joint (prismatic, 0.0–0.8m Z) + lift_link to mecanum URDF
- Sensor mounts (IMU, laser, depth camera) moved to lift_link
- Sensor macros now accept configurable parent_link parameter
- Replaced gz-sim plugins with gazebo_ros2_control hardware interface
- IMU plugin: gz-sim-imu-system → libgazebo_ros_imu_sensor.so

Controllers:
- mecanum_drive_controller: mecanum wheel drive (odom + tf)
- lift_controller: position_controllers/JointGroupPositionController
- joint_state_broadcaster: publishes all joint states
- controller_manager YAML at linorobot2_gazebo/config/

Launch (gazebo_classic.launch.py):
- robot_state_publisher → spawn_entity → controller spawners (timed)
- Controller load order: joint_state_broadcaster → mecanum → lift

Spawning (item_spawner.py):
- Z_CLEARANCE=0.05m: spawn above shelf surface, gravity settles
- Prevents physics explosion from collision mesh overlap on multi-level shelves

Dependencies installed:
- ros-humble-gazebo-ros2-control, ros-humble-mecanum-drive-controller
- ros-humble-position-controllers, ros-humble-joint-state-broadcaster

Co-Authored-By: Claude Opus 4.7 <noreply@anthropic.com>

File: src/linorobot2_description/urdf/robots/mecanum.urdf.xacro (robot description, xacro)
@@ -4,9 +4,12 @@
   <xacro:include filename="$(find linorobot2_description)/urdf/mech/base.urdf.xacro" />
   <xacro:include filename="$(find linorobot2_description)/urdf/mech/mecanum_wheel.urdf.xacro" />
+  <xacro:include filename="$(find linorobot2_description)/urdf/mech/lift.urdf.xacro" />
   <xacro:include filename="$(find linorobot2_description)/urdf/sensors/plugins.urdf.xacro" />
   <xacro:include filename="$(find linorobot2_description)/urdf/sensors/imu.urdf.xacro" />
   <xacro:include filename="$(find linorobot2_description)/urdf/sensors/generic_laser.urdf.xacro" />
   <xacro:include filename="$(find linorobot2_description)/urdf/sensors/depth_sensor.urdf.xacro" />
-  <xacro:include filename="$(find linorobot2_description)/urdf/controllers/omni_drive.urdf.xacro" />
+  <!-- ros2_control plugin replaces gz-sim omni_drive_controller for Gazebo Classic -->
+  <xacro:include filename="$(find linorobot2_description)/urdf/controllers/gazebo_ros2_control.urdf.xacro" />
+  <!-- Chassis base -->
   <xacro:base
     length="${base_length}"
@@ -18,4 +21,5 @@
     mesh_file="${base_mesh_file}"
   />
+  <!-- 4x Mecanum wheels -->
   <xacro:mecanum_wheel
     side="front_left"
@@ -58,15 +62,17 @@
     mesh_file="${wheel_mesh_file}"
   />
-  <xacro:imu/>
-  <xacro:generic_laser>
+  <!-- Prismatic lift mechanism (base_link → lift_link, 0.0–0.8m Z range) -->
+  <xacro:lift_mechanism base_length="${base_length}" />
+  <!-- Sensors mounted on lift_link for multi-level scanning -->
+  <xacro:imu parent_link="lift_link">
+    <origin xyz="0 0 0.05" rpy="0 0 0"/>
+  </xacro:imu>
+  <xacro:generic_laser parent_link="lift_link">
     <xacro:insert_block name="laser_pose" />
   </xacro:generic_laser>
-  <xacro:depth_sensor>
+  <xacro:depth_sensor parent_link="lift_link">
     <xacro:insert_block name="depth_sensor_pose" />
   </xacro:depth_sensor>
-  <xacro:omni_drive_controller
-    wheel_separation="${wheel_pos_y * 2}"
-    wheel_base="${wheel_pos_x * 2}"
-    wheel_radius="${wheel_radius}"
-  />
+  <!-- gazebo_ros2_control plugin (Gazebo Classic) -->
+  <xacro:gazebo_ros2_control_plugin />
 </robot>

File: src/linorobot2_description/urdf/sensors/depth_sensor.urdf.xacro (robot description, xacro)
@@ -1,5 +1,5 @@
 <robot xmlns:xacro="http://ros.org/wiki/xacro">
   <xacro:property name="M_PI" value="3.1415926535897931" />
-  <xacro:macro name="depth_sensor" params="*origin">
+  <xacro:macro name="depth_sensor" params="parent_link:=base_link *origin">
     <link name="camera_link">
       <visual>
@@ -7,5 +7,4 @@
         <geometry>
           <box size="0.030 0.124 0.030"/>
-          <!-- <mesh filename="" scale="0.001 0.001 0.001"/> -->
         </geometry>
         <material name="red">
@@ -36,7 +35,7 @@
         </material>
       </visual>
-    </gazebo>rgb(213,28,40)
-    <joint name="camera_to_base_link" type="fixed">
-      <parent link="base_link"/>
+    </gazebo>
+    <joint name="camera_joint" type="fixed">
+      <parent link="${parent_link}"/>
       <child link="camera_link"/>
       <xacro:insert_block name="origin" />

File: src/linorobot2_description/urdf/sensors/generic_laser.urdf.xacro (robot description, xacro)
@@ -2,5 +2,5 @@
 <robot xmlns:xacro="http://ros.org/wiki/xacro">
   <xacro:include filename="$(find linorobot2_description)/urdf/sensors/laser.urdf.xacro" />
-  <xacro:macro name="generic_laser" params="*origin">
+  <xacro:macro name="generic_laser" params="*origin parent_link:=base_link">
     <xacro:laser
       update_rate="10"
@@ -12,9 +12,10 @@
       frame_id="laser"
       topic_name="scan"
+      parent_link="${parent_link}"
     >
       <xacro:insert_block name="origin" />
     </xacro:laser>
   </xacro:macro>
-  <xacro:macro name="generic_base_laser" params="*origin">
+  <xacro:macro name="generic_base_laser" params="*origin parent_link:=base_link">
     <xacro:laser
       update_rate="10"
@@ -26,4 +27,5 @@
       frame_id="base_laser"
       topic_name="base/scan"
+      parent_link="${parent_link}"
     >
       <xacro:insert_block name="origin" />

File: src/linorobot2_description/urdf/sensors/imu.urdf.xacro (robot description, xacro)
@@ -1,12 +1,18 @@
 <robot xmlns:xacro="http://ros.org/wiki/xacro">
-  <xacro:macro name="imu">
+  <xacro:macro name="imu" params="parent_link:=base_link *origin">
     <link name="imu_link"/>
-    <joint name="imu_to_base_link" type="fixed">
-      <parent link="base_link"/>
+    <joint name="imu_joint" type="fixed">
+      <parent link="${parent_link}"/>
       <child link="imu_link"/>
-      <origin xyz="0 0 0" rpy="0 0 0"/>
+      <xacro:insert_block name="origin" />
     </joint>
     <gazebo>
-      <plugin filename="gz-sim-imu-system" name="gz::sim::systems::Imu">
+      <plugin filename="libgazebo_ros_imu_sensor.so"
+              name="gazebo_ros_imu_sensor">
+        <ros>
+          <namespace>/</namespace>
+          <remapping>~/out:=imu/data</remapping>
+        </ros>
+        <initial_orientation_as_reference>false</initial_orientation_as_reference>
       </plugin>
     </gazebo>

File: src/linorobot2_description/urdf/sensors/laser.urdf.xacro (robot description, xacro)
@@ -1,5 +1,5 @@
 <robot xmlns:xacro="http://ros.org/wiki/xacro">
   <xacro:property name="M_PI" value="3.1415926535897931" />
-  <xacro:macro name="laser" params="*origin update_rate ray_count min_angle max_angle min_range max_range frame_id topic_name">
+  <xacro:macro name="laser" params="*origin update_rate ray_count min_angle max_angle min_range max_range frame_id topic_name parent_link:=base_link">
     <link name="${frame_id}">
       <visual>
@@ -36,6 +36,6 @@
       </visual>
     </gazebo>
-    <joint name="${frame_id}_to_base_link" type="fixed">
-      <parent link="base_link"/>
+    <joint name="${frame_id}_joint" type="fixed">
+      <parent link="${parent_link}"/>
       <child link="${frame_id}"/>
       <xacro:insert_block name="origin" />
