Commit message: QA fix: optical frame rotation + depth encoding + calibration probe
URDF fix (depth_sensor.urdf.xacro):
- camera_depth_joint: rpy="0 0 0" → rpy="-1.570796 0 -1.570796"
  (REP 103: Z-forward optical axis, X-right, Y-down)
  Without this, TF2 projects depth to Z-up (ceiling/floor) instead of forward.

vision_node.py depth hardening:
- Replaced dtype-based depth conversion with msg.encoding-based logic
- Handles: 32FC1/32FC2 (metres), 16UC1/16UC2 (mm→m), mono16 (mm→m), mono8 (normalised)

calibration_check.py: new spatial accuracy probe
- Subscribes /target_object (PointStamped), computes Euclidean error
- Configurable ground-truth via ROS params (truth_x, truth_y, truth_z)

Co-Authored-By: Claude Opus 4.7 <noreply@anthropic.com>

File: src/linorobot2_description/urdf/sensors/depth_sensor.urdf.xacro (robot description, xacro)
@@ -41,7 +41,8 @@
       <xacro:insert_block name="origin" />
     </joint>
+    <!-- REP 103 optical frame: Z-forward (out of lens), X-right, Y-down -->
     <link name="camera_depth_link"/>
     <joint name="camera_depth_joint" type="fixed">
-      <origin xyz="0 0 0" rpy="0 0 0"/>
+      <origin xyz="0 0 0" rpy="-1.570796 0 -1.570796"/>
       <parent link="camera_link"/>
       <child link="camera_depth_link"/>
